File: Flight-Computer.kicad_sch (KiCad schematic)
At the start: 2 parts, among them U1 SX1262IMLTRT

Commit message: Updated schematic with LoRa and GPS module designs
Parts:
- removed L1: L, symbol Device:L
- removed U1: SX1262IMLTRT, Package_DFN_QFN:QFN-24-1EP_4x4mm_P0.5mm_EP2.6x2.6mm, symbol RF:SX1262IMLTRT
Other:
- added sheet GPS (GPS.kicad_sch)
- added sheet LoRa (LoRa.kicad_sch)
- note added: "Hierarchical modules for RF click into them!"

Commit message: Schematics for LoRa, GPS and power
Other:
- added sheet Buck Converter (DCDC.kicad_sch)
